File: Schematics/68hc11/68hc11.kicad_pcb (KiCad board)
At the start: 2 copper layers, 268.6 x 177.2 mm, 50 parts, among them J1 USB3076-30-A, J2 DB9_Female, J3 Conn_01x10_Male, J4 Conn_01x10_Male, J5 Conn_01x10_Male, J6 Conn_01x10_Male, J7 Conn_01x10_Male, SW1 Reset, U1 MC68HC11A1CC-PLLC, U10 MCP100-270D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

Commit message: Restarting the board layout
Parts:
- R1: footprint Resistor_THT:R_Axial_DIN0204_L3.6mm_D1.6mm_P7.62mm_Horizontal -> Resistor_THT:R_Axial_DIN0204_L3.6mm_D1.6mm_P5.08mm_Horizontal
- R2: footprint Resistor_THT:R_Axial_DIN0309_L9.0mm_D3.2mm_P12.70mm_Horizontal -> Resistor_THT:R_Axial_DIN0204_L3.6mm_D1.6mm_P5.08mm_Horizontal
- moved J3 340.6 mm to (-97.0, 28.3)
- moved J4 327.1 mm to (-92.5, 28.3)
- moved U2 316.7 mm to (-107.0, -24.3), turned to 0 degrees
- moved J7 292.4 mm to (-101.7, 28.3), turned to 0 degrees
- moved J6 282.1 mm to (-18.1, -24.1), turned to 0 degrees
- moved C19 272.9 mm to (-31.5, 36.1)
- moved J5 270.5 mm to (-106.2, 28.3), turned to 0 degrees
- moved U14 264.5 mm to (-3.35, -24.3)
- moved C21 263.2 mm to (-50.2, 48.9)
- moved C18 253.0 mm to (-35.2, 44.1)
- moved C2 253.0 mm to (-44.5, 47.2)
- moved U15 252.2 mm to (-20.6, 25.0)
- moved RN1 247.3 mm to (-88.0, 50.1)
- moved U12 243.5 mm to (-31.4, 17.0)
- moved U11 242.5 mm to (-42.3, 22.1)
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Connections:
- C10 pad 2: unconnected-(C10-Pad2) -> GND
- C17 pad 2: unconnected-(C17-Pad2) -> GND
- C18 pad 2: unconnected-(C18-Pad2) -> GND
- C19 pad 2: unconnected-(C19-Pad2) -> GND
- C20 pad 2: unconnected-(C20-Pad2) -> GND
- C21 pad 2: unconnected-(C21-Pad2) -> GND
- J3 pad 1: GND -> VCC
- J3 pad 10: unconnected-(J3-Pad10) -> GND
- J4 pad 1: VCC -> /VRL
- J4 pad 10: unconnected-(J4-Pad10) -> /VRH
- J4 pad 2: /PE0 -> unconnected-(J4-Pad2)
- U2 pad 37: unconnected-(U2-Pad37) -> /*IRQ
- U2 pad 38: unconnected-(U2-Pad38) -> /*IRQ
- U8 pad 20: unconnected-(U8-Pad20) -> /*RAM
- U8 pad 27: unconnected-(U8-Pad27) -> /R/*W
Routing:
- net GND: track 796.0 -> 0.00 mm, vias 3 -> 0
- net VCC: track 645.4 -> 0.00 mm, vias 1 -> 0
- net /*RESET: track 216.8 -> 0.00 mm, vias 3 -> 0
- net /D7: track 196.6 -> 0.00 mm, vias 1 -> 0
- net /R/*W: track 196.2 -> 0.00 mm, vias 3 -> 0
- net /D0: track 177.6 -> 0.00 mm
- net /D1: track 177.2 -> 0.00 mm, vias 1 -> 0
- net /D2: track 175.8 -> 0.00 mm
- net /D3: track 175.6 -> 0.00 mm
- net /D6: track 170.4 -> 0.00 mm
- net /D5: track 170.2 -> 0.00 mm
- net /D4: track 164.2 -> 0.00 mm
- net /A0: track 158.6 -> 0.00 mm, vias 2 -> 0
- net /A12: track 153.7 -> 0.00 mm, vias 3 -> 0
- net /TxD: track 153.4 -> 0.00 mm, vias 1 -> 0
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Other:
- board size 268.6 x 177.2 mm -> 224.5 x 119.5 mm
